Commit message: lidar not working atm

File: ros2/src/my_robot_description/urdf/robot.urdf.xacro (robot description, xacro)
@@ -1,51 +1,83 @@
 <?xml version="1.0"?>
-<robot name="my_robot" xmlns:xacro="http://www.ros.org/wiki/xacro">
-    <xacro:property name="wheel_radius" value="0.0425" />  <xacro:property name="wheel_base" value="0.15" />      <xacro:property name="base_width" value="0.25" />      <xacro:property name="base_length" value="0.30" />
-    <xacro:property name="base_height" value="0.05" />
-    <link name="base_link">
-        <visual>
-            <geometry>
-                <box size="${base_length} ${base_width} ${base_height}" />
-            </geometry>
-            <origin xyz="0 0 ${base_height/2}" rpy="0 0 0" />
-            <material name="blue">
-                <color rgba="0.1 0.1 0.8 1.0"/>
-            </material>
+<robot xmlns:xacro="http://www.ros.org/wiki/xacro" name="my_bot">
+  <xacro:property name="M_PI" value="3.1415926535897931" />
+  <xacro:property name="base_radius" value="0.2"/>
+  <xacro:property name="wheel_radius" value="0.05"/>
+  <xacro:property name="wheel_width"  value="0.02"/>
+  <xacro:property name="wheel_sep"    value="0.35"/>
+  <xacro:property name="wheel_x_offset" value="-0.02"/>
+  <xacro:property name="wheel_y_offset" value="0.19"/>
+  <xacro:property name="caster_radius" value="0.045"/>
+  <xacro:property name="caster_x_offset" value="0.18"/>
+  <material name="blue">
+    <color rgba="0.0 0.3 0.8 1.0"/>
+  </material>
+  <xacro:macro name="inertial_box" params="mass x y z">
+    <inertial>
+      <mass value="${mass}"/>
+      <origin xyz="0 0 0"/>
+      <inertia
+        ixx="${mass/12.0 * (y*y + z*z)}"
+        iyy="${mass/12.0 * (x*x + z*z)}"
+        izz="${mass/12.0 * (x*x + y*y)}"
+        ixy="0" ixz="0" iyz="0"/>
+    </inertial>
+  </xacro:macro>
+  <link name="base_link">
+    </link>
+  <link name="imu_link"/>
+  <joint name="imu_joint" type="fixed">
+    <parent link="base_link"/>
+    <child link="imu_link"/>
+    <origin xyz="0 0 0.15"/>
+  </joint>
+  <link name="lidar_link">
+    </link>
+  <joint name="lidar_joint" type="fixed">
+    <parent link="base_link"/>
+    <child link="lidar_link"/>
+    <origin xyz="0 0 0.18"/>
+  </joint>
+  <xacro:macro name="wheel" params="name y">
+    <link name="${name}">
+      <visual>
+        <origin xyz="0 0 0" rpy="0 ${M_PI/2} 0"/> <geometry>
+          <cylinder radius="${wheel_radius}" length="${wheel_width}"/>
+        </geometry>
+        <material name="dark"/>
         </visual>
-        <inertial>
-            <mass value="5.0" />
-            <inertia ixx="0.02" ixy="0.0" ixz="0.0" iyy="0.02" iyz="0.0" izz="0.02" />
-        </inertial>
+      <collision>
+        <origin xyz="0 0 0" rpy="0 ${M_PI/2} 0"/>
+        <geometry>
+          <cylinder radius="${wheel_radius}" length="${wheel_width}"/>
+        </geometry>
+      </collision>
+      <inertial>
+        <mass value="0.5"/>
+        <origin xyz="0 0 0"/>
+        <inertia
+          ixx="1e-3" iyy="1e-3" izz="1e-3"
+          ixy="0" ixz="0" iyz="0"/>
+      </inertial>
     </link>
-    <link name="left_wheel_link">
-        <visual>
-            <geometry>
-                <cylinder radius="${wheel_radius}" length="0.02" />
-            </geometry>
-            <origin xyz="0 0 0" rpy="${-M_PI/2} 0 0" />
-            <material name="black"/>
-        </visual>
+    <joint name="${name}_joint" type="continuous">
+      <parent link="base_link"/>
+      <child link="${name}"/>
+      <origin
+        xyz="${wheel_x_offset} ${y} ${wheel_radius}"
+        rpy="0 0 0"/>
+      <axis xyz="0 1 0"/>
+    </joint>
+  </xacro:macro>
+  <xacro:wheel name="wheel_left_link"  y="${ wheel_y_offset }"/>
+  <xacro:wheel name="wheel_right_link" y="${-wheel_y_offset }"/>
+  <link name="caster_link">
     </link>
-    <joint name="left_wheel_joint" type="continuous">
-        <parent link="base_link"/>
-        <child link="left_wheel_link"/>
-        <origin xyz="0 ${wheel_base/2} ${wheel_radius}" rpy="0 0 0" />
-        <axis xyz="0 1 0" />
-    </joint>
-    <link name="right_wheel_link">
-        </link>
-    <joint name="right_wheel_joint" type="continuous">
-        <parent link="base_link"/>
-        <child link="right_wheel_link"/>
-        <origin xyz="0 ${-wheel_base/2} ${wheel_radius}" rpy="0 0 0" />
-        <axis xyz="0 1 0" />
-    </joint>
-    <xacro:include filename="sensors.urdf.xacro" />
-    <xacro:sensor_macro />
-    <link name="odom" />
-    <joint name="odom_joint" type="fixed">
-        <parent link="odom"/>
-        <child link="base_link"/>
-        <origin xyz="0 0 0" rpy="0 0 0"/>
-    </joint>
-</robot>
+  <joint name="caster_joint" type="fixed">
+    <parent link="base_link"/>
+    <child link="caster_link"/>
+    <origin
+      xyz="${caster_x_offset} 0 0"
+      rpy="0 0 0"/>
+  </joint>
+  </robot>
